File: subcircuits/SchematicSketchpad/SchematicSketchpad.sch (KiCad schematic (older format))
At the start: 14 parts, among them Q1 BFR193W, Q2 BFR193W

Commit message: Added band-pass filter to RF front-end.
Parts:
- added C?: 15p, symbol Device:C
- added C?: 6p8, symbol Device:C
- added L? (x2): 390n, symbol Device:L
- added L?: 33n, symbol Device:L
- added R6: 18, symbol Device:R
- C4: value 10n -> 6p8
- RL: value 10k -> 50
Connections:
- net GND: now also C?.2, L?.2
- net at Q2.2 (E), R5.1: now also R6.2; no longer C4.2
- net at C4.1: now also L?.1; no longer RL.1
- new net: C4.2, R6.1
- new net: C?.1, C?.2, L?.1, L?.2
- new net: L?.2, RL.1
- new net: C?.1, L?.1
Other:
- note added: "3rd order Chebyshev band-pass filter"
- note added: "Amplifier Rout = 50 Ohms"
- note added: "Bandwidth (-3dB): 80 MHz to 120 MHz"
- note added: "Pass-band gain of matching circuit and filter circuit cancel.\nTotal gain is therefore 20dB in pass-band. (Assuming 50 Ohm load)"
- note added: "RF Matching, RF Amplifier, and Pass-Band RF Filter"
- note removed: "RF Matching and Amplifier"
- note removed: "Rout approx. = 22 Ohms"
- moved on the sheet: ANT, C1, C2, C3, C4, L1, Q1, Q2, R1, R2, R3, R4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
